File: business card.sch (KiCad schematic (older format))
At the start: 5 parts, among them U1 NT3H1101_NT3H1201

Commit message: Added all traces
Parts:
- removed L1: 2.75uH, symbol Device:L
- C1: footprint Capacitor_SMD:C_0603_1608Metric_Pad1.05x0.95mm_HandSolder -> Capacitor_SMD:C_0805_2012Metric_Pad1.15x1.40mm_HandSolder
- D1: footprint (none) -> LED_SMD:LED_0805_2012Metric_Pad1.15x1.40mm_HandSolder
- R1: footprint Resistor_SMD:R_0603_1608Metric_Pad1.05x0.95mm_HandSolder -> Resistor_SMD:R_0805_2012Metric_Pad1.15x1.40mm_HandSolder
Connections:
- net at U1.1 (LA): now also U1.8 (LB)
Changed lines of the file:
@@
 F 0 "R1" V 5950 5200 50  0000 L CNN
 F 1 "47ohm" V 6050 5200 50  0000 L CNN
-F 2 "Resistor_SMD:R_0603_1608Metric_Pad1.05x0.95mm_HandSolder" V 5780 5150 50  0001 C CNN
+F 2 "Resistor_SMD:R_0805_2012Metric_Pad1.15x1.40mm_HandSolder" V 5780 5150 50  0001 C CNN
 F 3 "~" H 5850 5150 50  0001 C CNN
 	1    5850 5150
@@
 F 0 "D1" H 5450 5050 50  0000 C CNN
 F 1 "LED" H 5450 4950 50  0000 C CNN
-F 2 "" H 5400 5150 50  0001 C CNN
+F 2 "LED_SMD:LED_0805_2012Metric_Pad1.15x1.40mm_HandSolder" H 5400 5150 50  0001 C CNN
 F 3 "~" H 5400 5150 50  0001 C CNN
 	1    5400 5150
-	1    0    0    -1
-$EndComp
-$Comp
-L Device:L L1
-U 1 1 5DB27CDD
-P 6300 3750
-F 0 "L1" H 6352 3796 50  0000 L CNN
-F 1 "2.75uH" H 6352 3705 50  0000 L CNN
-F 2 "" H 6300 3750 50  0001 C CNN
-F 3 "~" H 6300 3750 50  0001 C CNN
-	1    6300 3750
 	1    0    0    -1
 $EndComp
@@
 Wire Wire Line
 	5100 3500 6300 3500
-Wire Wire Line
-	6300 3500 6300 3600
 Wire Wire Line
 	6300 3900 6050 3900
@@
 Wire Wire Line
 	6300 4750 6300 4200
+Wire Wire Line
+	6300 5150 6300 4750
+Connection ~ 6300 4750
+Wire Wire Line
+	5100 5150 5100 4750
+Connection ~ 5100 4750
 $Comp
 L pspice:CAP C1
@@
 F 0 "C1" V 5800 4850 50  0000 L CNN
 F 1 "440nF" V 5900 4850 50  0000 L CNN
-F 2 "Capacitor_SMD:C_0603_1608Metric_Pad1.05x0.95mm_HandSolder" H 5700 4750 50  0001 C CNN
+F 2 "Capacitor_SMD:C_0805_2012Metric_Pad1.15x1.40mm_HandSolder" H 5700 4750 50  0001 C CNN
 F 3 "~" H 5700 4750 50  0001 C CNN
 	1    5700 4750
@@
 $EndComp
 Wire Wire Line
-	6300 5150 6300 4750
-Connection ~ 6300 4750
-Wire Wire Line
-	5100 5150 5100 4750
-Connection ~ 5100 4750
+	6300 3500 6300 3900
 $EndSCHEMATC
